File: PLL.kicad_sch (KiCad schematic)
At the start: 41 parts, among them J1 Center Pin, J2 Conn_01x01_Pin, J3 Conn_01x01_Pin, J4 Conn_01x01_Pin, M1 BS170, Q1 PN2907_PNP, Q3 P2N2222A_NPN, SW2 SW_SPDT, U2 74HC74, U3 LM324, U4 74HCT14N

Commit message: PCB design start
Parts:
- removed A1, A2, A3: LM324, symbol Amplifier_Operational:LM324
- removed A4, N1, N2, N3, N4: 74HC00, symbol 74xx:74HC00
- removed D1, D3, D5: 74HC74, symbol 74xx:74HC74
- removed unit 3 of D2
- removed unit 2 of D2
- removed M1: BS170, Package_TO_SOT_THT:TO-92_Inline, symbol Transistor_FET:BS170
- removed SW2: SW_SPDT, symbol Switch:SW_SPDT
- added J10: VpfdB2_tp, Connector_PinHeader_2.54mm:PinHeader_1x01_P2.54mm_Vertical, symbol Connector:Conn_01x01_Pin
- added J11: Vsq_tp, Connector_PinHeader_2.54mm:PinHeader_1x01_P2.54mm_Vertical, symbol Connector:Conn_01x01_Pin
- added J12: Vfb_tp, Connector_PinHeader_2.54mm:PinHeader_1x01_P2.54mm_Vertical, symbol Connector:Conn_01x01_Pin
- added J13: Ven_tp, Connector_PinHeader_2.54mm:PinHeader_1x01_P2.54mm_Vertical, symbol Connector:Conn_01x01_Pin
- added J14: Vref_tp, Connector_PinHeader_2.54mm:PinHeader_1x01_P2.54mm_Vertical, symbol Connector:Conn_01x01_Pin
- added J5: Vcp, Connector_PinHeader_2.54mm:PinHeader_1x01_P2.54mm_Vertical, symbol Connector:Conn_01x01_Pin
- added J6: Vout, Connector_PinHeader_2.54mm:PinHeader_1x01_P2.54mm_Vertical, symbol Connector:Conn_01x01_Pin
- added J7: Vin, Connector_PinHeader_2.54mm:PinHeader_1x01_P2.54mm_Vertical, symbol Connector:Conn_01x01_Pin
- added J8: Vctrl, Connector_PinHeader_2.54mm:PinHeader_1x01_P2.54mm_Vertical, symbol Connector:Conn_01x01_Pin
- added J9: VpfdB1_tp, Connector_PinHeader_2.54mm:PinHeader_1x01_P2.54mm_Vertical, symbol Connector:Conn_01x01_Pin
- added PWR_CONN1: power_conn, Connector_PinHeader_2.54mm:PinHeader_1x02_P2.54mm_Vertical, symbol Connector:Conn_01x02_Pin
- added Q2: BS170, Package_TO_SOT_THT:TO-92_Inline, symbol Transistor_FET:BS170
- added SW1: SW_SPDT, Button_Switch_THT:SW_Slide-03_Wuerth-WS-SLTV_10x2.5x6.4_P2.54mm, symbol Switch:SW_Wuerth_450301014042
- added U1: 74HC74, Package_DIP:DIP-14_W7.62mm_Socket, symbol 74xx:74HC74
- added unit 1 of U2
- added unit 3 of U2
- added unit 1 of U3
- added unit 2 of U3
- added unit 3 of U3
- added U5: 74HC00, Package_DIP:DIP-14_W7.62mm_Socket, symbol 74xx:74HC00
- C1, C2, C3: footprint (none) -> Capacitor_THT:C_Disc_D7.5mm_W2.5mm_P5.00mm
- J1: value Center Pin -> Vout; footprint (none) -> Connector_PinHeader_2.54mm:PinHeader_1x01_P2.54mm_Vertical
- J2: value Conn_01x01_Pin -> M=1; footprint (none) -> Connector_PinHeader_2.54mm:PinHeader_1x01_P2.54mm_Vertical
- J3: value Conn_01x01_Pin -> M=2; footprint (none) -> Connector_PinHeader_2.54mm:PinHeader_1x01_P2.54mm_Vertical
- J4: value Conn_01x01_Pin -> M=4; footprint (none) -> Connector_PinHeader_2.54mm:PinHeader_1x01_P2.54mm_Vertical
- Q1: footprint (none) -> Package_TO_SOT_THT:TO-92_Inline
- Q3: value P2N2222A_NPN -> PN2222A_NPN; footprint (none) -> Package_TO_SOT_THT:TO-92_Inline
- R1, R10, R11, R12, R2, R3, R4, R5, R6, R7, R8, R9: footprint (none) -> Resistor_THT:R_Axial_DIN0204_L3.6mm_D1.6mm_P7.62mm_Horizontal
- U2, U3, U4: footprint (none) -> Package_DIP:DIP-14_W7.62mm_Socket
Connections:
- net Earth: now also U4.7 (GND), PWR_CONN1.2 (Pin_2), Q2.1 (S), SW1.2 (C), U1.7 (GND), U2.7 (GND), U5.7 (GND); no longer U4.3 (GND)
- net VCC: now also U2.13 (~{R}), U4.14 (VCC), PWR_CONN1.1 (Pin_1), SW1.3 (A), U1.10 (~{S}), U1.12 (D), U1.14 (VCC), U1.2 (D), U1.4 (~{S}), U2.1 (~{R}), U2.14 (VCC), U2.4 (~{S}), U5.14 (VCC); no longer U2.12 (D), U4.5 (VCC)
- net at J2.1 (Pin_1): now also J12.1 (Pin_1), U1.11 (C), U2.5 (Q); no longer U2.11 (C)
- net at R4.1, R5.2: now also J8.1 (Pin_1), U3.8, U3.9 (-)
- net at R5.1, R6.2: now also U3.5 (+)
- net at C1.1, R4.2, R7.1: now also U3.6 (-)
- net at C1.2: now also U3.2 (-), U3.7
- net at Q1.1 (E): now also R10.2; no longer Q3.1 (C)
- net at Q1.3 (C): now also Q3.3 (C); no longer R10.2
- net at U2.8 (~{Q}): now also U2.12 (D)
- net at R11.1: now also J10.1 (Pin_1), U1.9 (Q), U5.12; no longer U2.9 (Q)
- net at R7.2: now also Q2.3 (D)
- net at J4.1 (Pin_1): now also U2.11 (C)
- net at J3.1 (Pin_1): now also U2.9 (Q), U2.3 (C)
- net at R12.1: now also J9.1 (Pin_1), U1.6 (~{Q})
- net at R1.1, R2.2, R3.1: now also U3.3 (+)
- net at R9.1: now also Q3.1 (E); no longer Q3.3 (E)
- net Vcp: no longer names the net of C3.2, R8.1
- net Vcp: now also J5.1 (Pin_1), U3.10 (+)
- net Vout: no longer names the net of J1.1 (Pin_1)
- net Vout: now also U4.2, J6.1 (Pin_1); no longer U4.4
- net Vsq: no longer names the net of R3.2
- net Vsq: now also U4.1 (NC), Q2.2 (G), U3.1; no longer U4.2
- new net: U5.10, U5.11, U5.9
- new net: U5.4, U5.5, U5.8
- new net: U1.5 (Q), U5.13
- new net: U2.2 (D), U2.6 (~{Q})
- new net: J7.1 (Pin_1), U5.1
- new net: J13.1 (Pin_1), SW1.1 (B), U5.2
- new net: J14.1 (Pin_1), U1.3 (C), U5.3
- new net: U1.1 (~{R}), U1.13 (~{R}), U5.6

Commit message: add LED indicator
Parts:
- added D5: LED, LED_THT:LED_D5.0mm, symbol Device:LED
- added R13: 330, Resistor_THT:R_Axial_DIN0204_L3.6mm_D1.6mm_P7.62mm_Horizontal, symbol Device:R_US
- J10: value VpfdB2_tp -> VpfdB2
- J11: value Vsq_tp -> Vsq
- J12: value Vfb_tp -> Vfb
- J13: value Ven_tp -> Ven
- J14: value Vref_tp -> Vref
- J9: value VpfdB1_tp -> VpfdB1
- renumbered PWR_CONN1 to PWR_HEADER
Connections:
- net Earth: now also D5.1 (K)
- net VCC: now also R13.1
- new net: D5.2 (A), R13.2
Changed lines of the file:
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@@
 	)
 	(junction
+		(at 88.9 54.61)
+		(diameter 0)
+		(color 0 0 0 0)
+	)
+	(junction
 		(at 161.29 124.46)
 		(diameter 0)
@@
 	)
 	(junction
+		(at 88.9 74.93)
+		(diameter 0)
+		(color 0 0 0 0)
+	)
+	(junction
 		(at 190.3636 130.81)
 		(diameter 0)
@@
 	(wire
 		(pts
+			(xy 88.9 54.61) (xy 100.33 54.61)
+		)
+		(stroke
+			(width 0)
+			(type default)
+		)
+	)
+	(wire
+		(pts
 			(xy 298.45 133.35) (xy 298.45 132.08)
 		)
@@
 	(wire
 		(pts
+			(xy 100.33 74.93) (xy 88.9 74.93)
+		)
+		(stroke
+			(width 0)
+			(type default)
+		)
+	)
+	(wire
+		(pts
 			(xy 349.25 104.14) (xy 353.06 104.14)
 		)
@@
 	(wire
 		(pts
+			(xy 100.33 64.77) (xy 100.33 66.04)
+		)
+		(stroke
+			(width 0)
+			(type default)
+		)
+	)
+	(wire
+		(pts
 			(xy 190.3636 130.81) (xy 195.5771 130.81)
 		)
@@
 	(wire
 		(pts
+			(xy 100.33 73.66) (xy 100.33 74.93)
+		)
+		(stroke
+			(width 0)
+			(type default)
+		)
+	)
+	(wire
+		(pts
 			(xy 393.7 118.11) (xy 391.16 118.11)
 		)
@@
 	(wire
 		(pts
+			(xy 100.33 54.61) (xy 100.33 57.15)
+		)
+		(stroke
+			(width 0)
+			(type default)
+		)
+	)
+	(wire
+		(pts
 			(xy 327.66 115.57) (xy 327.66 123.19)
 		)
@@
 		(on_board yes)
 		(dnp no)
-		(property "Reference" "PWR_CONN1"
+		(property "Reference" "PWR_HEADER"
 			(at 26.924 59.436 0)
 			(effects
@@
 			(project ""
 				(path "/ac247623-a02d-4cc5-be05-0b11086d5480"
-					(reference "PWR_CONN1")
+					(reference "PWR_HEADER")
 					(unit 1)
 				)
@@
 		(dnp no)
 		(property "Reference" "J9"
-			(at 187.96 119.38 90)
+			(at 189.23 114.046 90)
 			(effects
 				(font
@@
 			)
 		)
-		(property "Value" "VpfdB1_tp"
+		(property "Value" "VpfdB1"
 			(at 188.976 121.666 90)
 			(effects
@@
 	)
 	(symbol
+		(lib_id "Device:LED")
+		(at 100.33 69.85 90)
+		(unit 1)
+		(exclude_from_sim no)
+		(in_bom yes)
+		(on_board yes)
+		(dnp no)
+		(fields_autoplaced yes)
+		(property "Reference" "D5"
+			(at 104.14 70.1674 90)
+			(effects
+				(font
+					(size 1.27 1.27)
+				)
+				(justify right)
+			)
+		)
+		(property "Value" "LED"
+			(at 104.14 72.7074 90)
+			(effects
+				(font
+					(size 1.27 1.27)
+				)
+				(justify right)
+			)
+		)
+		(property "Footprint" "LED_THT:LED_D5.0mm"
+			(at 100.33 69.85 0)
+			(effects
+				(font
+					(size 1.27 1.27)
+				)
+				(hide yes)
+			)
+		)
+		(property "Datasheet" "~"
+			(at 100.33 69.85 0)
+			(effects
+				(font
+					(size 1.27 1.27)
+				)
+				(hide yes)
+			)
+		)
+		(property "Description" "Light emitting diode"
+			(at 100.33 69.85 0)
+			(effects
+				(font
+					(size 1.27 1.27)
+				)
+				(hide yes)
+			)
+		)
+		(property "Sim.Pins" "1=K 2=A"
+			(at 100.33 69.85 0)
+			(effects
+				(font
+					(size 1.27 1.27)
+				)
+				(hide yes)
+			)
+		)
+		(pin "1"
+		)
+		(pin "2"
+		)
+		(instances
+			(project ""
+				(path "/ac247623-a02d-4cc5-be05-0b11086d5480"
+					(reference "D5")
+					(unit 1)
+				)
+			)
+		)
+	)
+	(symbol
 		(lib_id "power:VCC")
 		(at 327.66 104.14 0)
@@
 			)
 		)
-		(property "Value" "Vsq_tp"
+		(property "Value" "Vsq"
 			(at 355.346 124.206 90)
 			(effects
@@
 	)
 	(symbol
+		(lib_id "Device:R_US")
+		(at 100.33 60.96 0)
+		(unit 1)
+		(exclude_from_sim no)
+		(in_bom yes)
+		(on_board yes)
+		(dnp no)
+		(property "Reference" "R13"
+			(at 105.41 60.706 90)
+			(effects
+				(font
+					(size 1.27 1.27)
+				)
+			)
+		)
+		(property "Value" "330"
+			(at 102.87 60.706 90)
+			(effects
+				(font
+					(size 1.27 1.27)
+				)
+			)
+		)
+		(property "Footprint" "Resistor_THT:R_Axial_DIN0204_L3.6mm_D1.6mm_P7.62mm_Horizontal"
+			(at 101.346 61.214 90)
+			(effects
+				(font
+					(size 1.27 1.27)
+				)
+				(hide yes)
+			)
+		)
+		(property "Datasheet" "~"
+			(at 100.33 60.96 0)
+			(effects
+				(font
+					(size 1.27 1.27)
+				)
+				(hide yes)
+			)
+		)
+		(property "Description" "Resistor, US symbol"
+			(at 100.33 60.96 0)
+			(effects
+				(font
+					(size 1.27 1.27)
+				)
+				(hide yes)
+			)
+		)
+		(pin "2"
+		)
+		(pin "1"
+		)
+		(instances
+			(project "PLL"
+				(path "/ac247623-a02d-4cc5-be05-0b11086d5480"
+					(reference "R13")
+					(unit 1)
+				)
+			)
+		)
+	)
+	(symbol
 		(lib_id "Connector:Conn_01x01_Pin")
 		(at 226.06 205.74 90)
@@
 			)
 		)
-		(property "Value" "Vfb_tp"
+		(property "Value" "Vfb"
 			(at 185.166 186.436 90)
 			(effects
@@
 			)
 		)
-		(property "Value" "Vref_tp"
+		(property "Value" "Vref"
 			(at 100.076 119.126 90)
 			(effects
@@
 		(dnp no)
 		(property "Reference" "J10"
-			(at 187.8236 134.62 90)
+			(at 188.214 129.794 90)
 			(effects
 				(font
@@
 			)
 		)
-		(property "Value" "VpfdB2_tp"
+		(property "Value" "VpfdB2"
 			(at 188.8396 136.906 90)
 			(effects
@@
 			)
 		)
-		(property "Value" "Ven_tp"
+		(property "Value" "Ven"
 			(at 78.486 121.666 90)
 			(effects

Commit message: Vsq connection fix
Parts:
- renumbered PWR_HEADER to PWR_HEADER1
Connections:
- net at Q2.2 (G), R3.2, U3.1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: now also J11.1 (Pin_1)
Changed lines of the file:
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@@
 	(generator "eeschema")
 	(generator_version "9.0")
-	(paper "A2")
+	(paper "A3")
 	(title_block
 		(title "PLL")
@@
 	)
 	(junction
+		(at 356.87 118.11)
+		(diameter 0)
+		(color 0 0 0 0)
+	)
+	(junction
 		(at 80.01 115.57)
 		(diameter 0)
@@
 	(wire
 		(pts
+			(xy 356.87 118.11) (xy 363.22 118.11)
+		)
+		(stroke
+			(width 0)
+			(type default)
+		)
+	)
+	(wire
+		(pts
 			(xy 215.9 200.66) (xy 198.12 200.66)
 		)
@@
 	(wire
 		(pts
-			(xy 353.06 118.11) (xy 363.22 118.11)
+			(xy 353.06 118.11) (xy 356.87 118.11)
 		)
 		(stroke
@@
 		(on_board yes)
 		(dnp no)
-		(property "Reference" "PWR_HEADER"
+		(property "Reference" "PWR_HEADER1"
 			(at 26.924 59.436 0)
 			(effects
@@
 			(project ""
 				(path "/ac247623-a02d-4cc5-be05-0b11086d5480"
-					(reference "PWR_HEADER")
+					(reference "PWR_HEADER1")
 					(unit 1)
 				)
@@
 				)
 				(justify left)
-				(hide yes)
 			)
 		)
